Commit message: updated mining_map

File: src/chassis_base_model/urdf/mecanum.xacro (robot description, xacro)
@@ -4,4 +4,5 @@
 <xacro:include filename="$(find mecanum_description)/urdf/mecanum.trans" />
 <xacro:include filename="$(find mecanum_description)/urdf/mecanum.gazebo" />
+<link name="world_map"/>
 <link name="base_link">
   <inertial>
@@ -184,4 +185,9 @@
   </collision>
 </link>
+<joint name="3d_free_move" type="planar">
+  <origin xyz="0 0 0" rpy="0 0 0"/>
+  <parent link="world_map"/>
+  <child link="base_link"/>
+</joint>
 <joint name="Rigid 47" type="fixed">
   <origin xyz="0.086916 0.106958 0.03048" rpy="0 0 0"/>
